File: RTC_Circuit/RTC_Circuit.sch (KiCad schematic (older format))
At the start: 3 parts, among them U1 DS3231M

Commit message: Added spectrometer, photodiode, and atmega to sch
Parts:
- added C? (x4): C_Small, symbol Device:C_Small
- added C?: CP_Small, symbol Device:CP_Small
- added C? (x2): CP1_Small, symbol Device:CP1_Small
- added R? (x2): R_10K, footprints:R_0805_OEM, symbol RTC_Circuit-rescue:R_10K-formula
- added R?: R, symbol Device:R
- added U?: ATmega32U4-MU, Package_DFN_QFN:QFN-44-1EP_7x7mm_P0.5mm_EP5.2x5.2mm, symbol MCU_Microchip_ATmega:ATmega32U4-MU
- added U?: DF12-20DS, symbol Custom:DF12-20DS
- added U?: S1336-44BQ, symbol Custom:S1336-44BQ
- added U?: S14739-20, symbol Custom:S14739-20
- added U?: LT1818, symbol Custom:LT1818
- R? (x2): symbol formula:R_10K -> RTC_Circuit-rescue:R_10K-formula
Connections:
- net labels added: 3.3V, 5V, GNDA, RX, TX
- wire segments 0 -> 47
- no-connect marks 0 -> 6
Other:
- note added: "Microcontroller"
- note added: "NSL Connector"
- note added: "Photodiode"
- note added: "Real Time Clock"
- note added: "Spectrometer"
- moved on the sheet: R?, U1

Commit message: Began writing code for electronics on Joe and Bill satellites
Parts:
- added D? (x3): LED, symbol Device:LED
- added J?: Conn_02x03_Counter_Clockwise, symbol Connector_Generic:Conn_02x03_Counter_Clockwise
- added R? (x3): R, symbol Device:R
- added R?: R_10K, footprints:R_0805_OEM, symbol RTC_Circuit-rescue:R_10K-formula
- added U?: MCP9700AT-HLT, Package_TO_SOT_SMD:SOT-353_SC-70-5, symbol Sensor_Temperature:MCP9700AT-HLT
- added U?: OPAMP, symbol pspice:OPAMP
Connections:
- net labels added: +5V, BUSY, CRYSTAL, EOS, MISO, MOSI, PHOV, RST, SCK, SDA, SQW, ST, TEMPV, Trig
- wire segments 47 -> 89
- no-connect marks 6 -> 8
Other:
- note added: "Programming Header"
- note added: "Programming LEDs"
- note added: "Temperature Sensor"
- moved on the sheet: C?, U?
