File: Circuitry/Burt/_autosave-Burt.sch (KiCad schematic (older format))
At the start: 52 parts

Commit message: motor driver
Parts:
- removed D?: D, symbol Device:D
- added R?: 18k, symbol Device:R_Small
- added R?: 10k, symbol Device:R_Small
Connections:
- net +BATT: now also U?.1 (OUTB); no longer M?.1 (+)
- net GNDA: now also U?.4 (OUTA), R?.2
- net at M?.2 (-): now also U?.3 (VDD)
- net at U?.2 (GND): now also M?.1 (+)
- net at U?.5 (VSET): now also R?.1, R?.2
- net at U?.6 (VREF): now also R?.1
- net IN2: now reaches U?.7 (IN1)
- net IN1: now reaches U?.8 (IN2)
Other:
- moved on the sheet: M?, U?
Changed lines of the file:
@@
 Connection ~ 1550 4275
+$Comp
+L Custom:A3908 U?
+U 1 1 5D5325EF
+P 2425 6525
+F 0 "U?" H 2425 6940 50  0000 C CNN
+F 1 "A3908" H 2425 6849 50  0000 C CNN
+F 2 "" H 1975 6375 50  0001 C CNN
+F 3 "" H 1975 6375 50  0001 C CNN
+	1    2425 6525
+	1    0    0    -1
+$EndComp
+$Comp
+L Device:R_Small R?
+U 1 1 5D538E55
+P 3000 6675
+F 0 "R?" H 3059 6721 50  0000 L CNN
+F 1 "18k" H 3059 6630 50  0000 L CNN
+F 2 "" H 3000 6675 50  0001 C CNN
+F 3 "~" H 3000 6675 50  0001 C CNN
+	1    3000 6675
+	1    0    0    -1
+$EndComp
+$Comp
+L Device:R_Small R?
+U 1 1 5D543F60
+P 3000 6975
+F 0 "R?" H 2850 6950 50  0000 L CNN
+F 1 "10k" H 2800 6875 50  0000 L CNN
+F 2 "" H 3000 6975 50  0001 C CNN
+F 3 "~" H 3000 6975 50  0001 C CNN
+	1    3000 6975
+	1    0    0    -1
+$EndComp
+$Comp
+L power:+BATT #PWR?
+U 1 1 5D545C7D
+P 1675 6375
+F 0 "#PWR?" H 1675 6225 50  0001 C CNN
+F 1 "+BATT" H 1690 6548 50  0000 C CNN
+F 2 "" H 1675 6375 50  0001 C CNN
+F 3 "" H 1675 6375 50  0001 C CNN
+	1    1675 6375
+	1    0    0    -1
+$EndComp
+Wire Wire Line
+	1675 6375 2075 6375
+Wire Wire Line
+	2775 6575 3000 6575
+Wire Wire Line
+	3000 6775 3000 6825
+Wire Wire Line
+	2775 6675 2775 6825
+Wire Wire Line
+	2775 6825 3000 6825
+Connection ~ 3000 6825
+Wire Wire Line
+	3000 6825 3000 6875
+$Comp
+L power:GNDA #PWR?
+U 1 1 5D559B0F
+P 2450 7175
+F 0 "#PWR?" H 2450 6925 50  0001 C CNN
+F 1 "GNDA" H 2455 7002 50  0000 C CNN
+F 2 "" H 2450 7175 50  0001 C CNN
+F 3 "" H 2450 7175 50  0001 C CNN
+	1    2450 7175
+	1    0    0    -1
+$EndComp
+Wire Wire Line
+	3000 7075 3000 7175
+Wire Wire Line
+	3000 7175 2450 7175
+Wire Wire Line
+	2075 6675 2075 7175
+Wire Wire Line
+	2075 7175 2450 7175
+Connection ~ 2450 7175
 $Comp
 L Motor:Motor_DC M?
 U 1 1 5D49D045
-P -275 4825
-F 0 "M?" H -117 4821 50  0000 L CNN
-F 1 "Motor_DC" H -117 4730 50  0000 L CNN
-F 2 "" H -275 4735 50  0001 C CNN
-F 3 "~" H -275 4735 50  0001 C CNN
-	1    -275 4825
+P 1650 6775
+F 0 "M?" V 1325 6800 50  0000 L CNN
+F 1 "Motor_DC" V 1425 6550 50  0000 L CNN
+F 2 "" H 1650 6685 50  0001 C CNN
+F 3 "~" H 1650 6685 50  0001 C CNN
+	1    1650 6775
 	1    0    0    -1
 $EndComp
+Text Label 3000 6375 0    50   ~ 0
+IN1
+Text Label 3000 6475 0    50   ~ 0
+IN2
 Wire Wire Line
-	-825 5125 -575 5125
-$Comp
-L Device:D D?
-U 1 1 5D4E1505
-P -575 4975
-F 0 "D?" V -621 5054 50  0000 L CNN
-F 1 "D" V -530 5054 50  0000 L CNN
-F 2 "" H -575 4975 50  0001 C CNN
-F 3 "~" H -575 4975 50  0001 C CNN
-	1    -575 4975
-	0    1    1    0
-$EndComp
-Connection ~ -575 5125
+	2775 6375 3000 6375
 Wire Wire Line
-	-575 5125 -275 5125
-$Comp
-L power:+BATT #PWR?
-U 1 1 5D504796
-P -275 3975
-F 0 "#PWR?" H -275 3825 50  0001 C CNN
-F 1 "+BATT" H -260 4148 50  0000 C CNN
-F 2 "" H -275 3975 50  0001 C CNN
-F 3 "" H -275 3975 50  0001 C CNN
-	1    -275 3975
-	1    0    0    -1
-$EndComp
+	2775 6475 3000 6475
 Wire Wire Line
-	-275 4625 -275 4575
+	2075 6475 1650 6475
 Wire Wire Line
-	-575 4825 -575 4575
+	1650 6475 1650 6575
 Wire Wire Line
-	-575 4575 -275 4575
-Connection ~ -275 4575
+	2075 6575 1875 6575
 Wire Wire Line
-	-275 3975 -275 4575
-$Comp
-L Custom:A3908 U?
-U 1 1 5D5325EF
-P -1525 5325
-F 0 "U?" H -1525 5740 50  0000 C CNN
-F 1 "A3908" H -1525 5649 50  0000 C CNN
-F 2 "" H -1975 5175 50  0001 C CNN
-F 3 "" H -1975 5175 50  0001 C CNN
-	1    -1525 5325
-	1    0    0    -1
-$EndComp
+	1875 6575 1875 7075
+Wire Wire Line
+	1875 7075 1650 7075
 $EndSCHEMATC
