File: Circuitry/Burt/Burt.sch (KiCad schematic (older format))
At the start: 29 parts

Commit message: Pinouts for sensors on burt and calc_state
Parts:
- removed R? (x4): R_10K, footprints:R_0805_OEM, symbol RTC_Circuit-rescue:R_10K-formula
- added R? (x4): R, symbol Device:R
Connections:
- net labels added: PHO1, PHO2, TEMP, VID
- net labels removed: PHOV, PHOV1, PHOV2
Changed lines of the file:
@@
 	10650 3450 10875 3450
 Text Label 10875 3450 0    50   ~ 0
-TEMPV
+TEMP
 Text Label 1550 5400 3    50   ~ 0
 TEMPV
@@
 Wire Wire Line
 	2000 1550 1750 1550
-$Comp
-L RTC_Circuit-rescue:R_10K-formula R?
-U 1 1 5D34875D
-P 1125 1075
-F 0 "R?" V 1225 1075 50  0000 L CNN
-F 1 "R_10K" V 1300 1075 50  0000 L CNN
-F 2 "footprints:R_0805_OEM" H 1055 1075 50  0001 C CNN
-F 3 "http://www.bourns.com/data/global/pdfs/CRS.pdf" H 1205 1075 50  0001 C CNN
-F 4 "DK" H 1125 1075 60  0001 C CNN "MFN"
-F 5 "CRS0805-FX-1002ELFCT-ND" H 1125 1075 60  0001 C CNN "MPN"
-F 6 "https://www.digikey.com/products/en?keywords=CRS0805-FX-1002ELFCT-ND" H 1605 1475 60  0001 C CNN "PurchasingLink"
-	1    1125 1075
-	0    -1   -1   0
-$EndComp
 $Comp
 L pspice:OPAMP U?
@@
 	1750 1750 1750 1950
 Text Label 825  1650 2    50   ~ 0
-PHOV1
+PHO1
 Text Label 10850 1950 0    50   ~ 0
-PHOV
+PHO1
 Wire Wire Line
 	10650 1950 10850 1950
@@
 	2000 2875 1750 2875
 $Comp
-L RTC_Circuit-rescue:R_10K-formula R?
-U 1 1 5D2A23E0
-P 1125 2400
-F 0 "R?" V 1225 2400 50  0000 L CNN
-F 1 "R_10K" V 1300 2400 50  0000 L CNN
-F 2 "footprints:R_0805_OEM" H 1055 2400 50  0001 C CNN
-F 3 "http://www.bourns.com/data/global/pdfs/CRS.pdf" H 1205 2400 50  0001 C CNN
-F 4 "DK" H 1125 2400 60  0001 C CNN "MFN"
-F 5 "CRS0805-FX-1002ELFCT-ND" H 1125 2400 60  0001 C CNN "MPN"
-F 6 "https://www.digikey.com/products/en?keywords=CRS0805-FX-1002ELFCT-ND" H 1605 2800 60  0001 C CNN "PurchasingLink"
-	1    1125 2400
-	0    -1   -1   0
-$EndComp
-$Comp
 L pspice:OPAMP U?
 U 1 1 5D2A23E6
@@
 	1750 3075 1750 3275
 Text Label 825  2975 2    50   ~ 0
-PHOV2
+PHO2
 $Comp
 L Custom:S1336-44BQ U?
@@
 Wire Wire Line
 	4175 1450 3925 1450
-$Comp
-L RTC_Circuit-rescue:R_10K-formula R?
-U 1 1 5D2AB627
-P 3300 975
-F 0 "R?" V 3400 975 50  0000 L CNN
-F 1 "R_10K" V 3475 975 50  0000 L CNN
-F 2 "footprints:R_0805_OEM" H 3230 975 50  0001 C CNN
-F 3 "http://www.bourns.com/data/global/pdfs/CRS.pdf" H 3380 975 50  0001 C CNN
-F 4 "DK" H 3300 975 60  0001 C CNN "MFN"
-F 5 "CRS0805-FX-1002ELFCT-ND" H 3300 975 60  0001 C CNN "MPN"
-F 6 "https://www.digikey.com/products/en?keywords=CRS0805-FX-1002ELFCT-ND" H 3780 1375 60  0001 C CNN "PurchasingLink"
-	1    3300 975
-	0    -1   -1   0
-$EndComp
 $Comp
 L pspice:OPAMP U?
@@
 	3925 1650 3925 1850
 Text Label 3000 1550 2    50   ~ 0
-PHOV2
+PHO2
 $Comp
 L Custom:S1336-44BQ U?
@@
 Wire Wire Line
 	4175 2800 3925 2800
-$Comp
-L RTC_Circuit-rescue:R_10K-formula R?
-U 1 1 5D16F477
-P 3300 2325
-F 0 "R?" V 3400 2325 50  0000 L CNN
-F 1 "R_10K" V 3475 2325 50  0000 L CNN
-F 2 "footprints:R_0805_OEM" H 3230 2325 50  0001 C CNN
-F 3 "http://www.bourns.com/data/global/pdfs/CRS.pdf" H 3380 2325 50  0001 C CNN
-F 4 "DK" H 3300 2325 60  0001 C CNN "MFN"
-F 5 "CRS0805-FX-1002ELFCT-ND" H 3300 2325 60  0001 C CNN "MPN"
-F 6 "https://www.digikey.com/products/en?keywords=CRS0805-FX-1002ELFCT-ND" H 3780 2725 60  0001 C CNN "PurchasingLink"
-	1    3300 2325
-	0    -1   -1   0
-$EndComp
 $Comp
 L pspice:OPAMP U?
@@
 	3925 3000 3925 3200
 Text Label 3000 2900 2    50   ~ 0
-PHOV2
+PHO2
 Wire Notes Line
 	525  525  4800 525
@@
 Wire Notes Line
 	4875 5900 4875 3675
+Text Label 8425 2900 0    50   ~ 0
+VID
+$Comp
+L Device:R R?
+U 1 1 5D302F96
+P 1125 1075
+F 0 "R?" V 918 1075 50  0000 C CNN
+F 1 "R" V 1009 1075 50  0000 C CNN
+F 2 "" V 1055 1075 50  0001 C CNN
+F 3 "~" H 1125 1075 50  0001 C CNN
+	1    1125 1075
+	0    1    1    0
+$EndComp
+$Comp
+L Device:R R?
+U 1 1 5D305A66
+P 3300 975
+F 0 "R?" V 3093 975 50  0000 C CNN
+F 1 "R" V 3184 975 50  0000 C CNN
+F 2 "" V 3230 975 50  0001 C CNN
+F 3 "~" H 3300 975 50  0001 C CNN
+	1    3300 975
+	0    1    1    0
+$EndComp
+$Comp
+L Device:R R?
+U 1 1 5D30B8FB
+P 3300 2325
+F 0 "R?" V 3093 2325 50  0000 C CNN
+F 1 "R" V 3184 2325 50  0000 C CNN
+F 2 "" V 3230 2325 50  0001 C CNN
+F 3 "~" H 3300 2325 50  0001 C CNN
+	1    3300 2325
+	0    1    1    0
+$EndComp
+$Comp
+L Device:R R?
+U 1 1 5D30ED97
+P 1125 2400
+F 0 "R?" V 918 2400 50  0000 C CNN
+F 1 "R" V 1009 2400 50  0000 C CNN
+F 2 "" V 1055 2400 50  0001 C CNN
+F 3 "~" H 1125 2400 50  0001 C CNN
+	1    1125 2400
+	0    1    1    0
+$EndComp
 $EndSCHEMATC

Commit message: bus sensor pins and additional circuitry
Parts:
- added C? (x2): C, symbol Device:C
- added C?: CP, symbol Device:CP
- added R?: R, symbol Device:R
Connections:
- net labels added: -5V, B1, B10, B2, B3, B4, B5, B6, B7, B8, B9, PHO3, PHO4, TRIG
- net labels removed: TEMPV
- wire segments 85 -> 103
Other:
- moved on the sheet: R?, U?
Changed lines of the file:
@@
 Text Label 9250 1750 2    50   ~ 0
 CRYSTAL
-Text Label 10875 3750 0    50   ~ 0
+Text Label 10850 2250 0    50   ~ 0
 SQW
 Wire Wire Line
@@
 Wire Wire Line
 	10650 3450 10875 3450
-Text Label 10875 3450 0    50   ~ 0
+Text Label 10850 2150 0    50   ~ 0
 TEMP
 Text Label 1550 5400 3    50   ~ 0
-TEMPV
+TEMP
 Wire Wire Line
 	1550 5175 1550 5400
@@
 	1750 3075 1750 3275
 Text Label 825  2975 2    50   ~ 0
-PHO2
+PHO3
 $Comp
 L Custom:S1336-44BQ U?
@@
 	3925 3000 3925 3200
 Text Label 3000 2900 2    50   ~ 0
-PHO2
+PHO4
 Wire Notes Line
 	525  525  4800 525
@@
 Wire Notes Line
 	8700 525  8700 3575
-Wire Notes Line
-	8700 3575 4875 3575
 Wire Notes Line
 	4875 3575 4875 525
@@
 	7200 2100 7700 2100
 NoConn ~ 7200 2000
-Wire Wire Line
-	8325 2900 8425 2900
-Connection ~ 8325 2900
-Wire Wire Line
-	8225 2900 8325 2900
-Wire Wire Line
-	8325 3475 8325 2900
-Wire Wire Line
-	7625 3475 8325 3475
-Wire Wire Line
-	7625 3000 7625 3475
 $Comp
 L power:GNDA #PWR?
 U 1 1 5D1F2D73
-P 7825 3200
-F 0 "#PWR?" H 7825 2950 50  0001 C CNN
-F 1 "GNDA" H 7830 3027 50  0000 C CNN
-F 2 "" H 7825 3200 50  0001 C CNN
-F 3 "" H 7825 3200 50  0001 C CNN
-	1    7825 3200
-	1    0    0    -1
-$EndComp
-Text Label 7825 2600 0    50   ~ 0
+P 6450 3450
+F 0 "#PWR?" H 6450 3200 50  0001 C CNN
+F 1 "GNDA" H 6275 3375 50  0000 C CNN
+F 2 "" H 6450 3450 50  0001 C CNN
+F 3 "" H 6450 3450 50  0001 C CNN
+	1    6450 3450
+	1    0    0    -1
+$EndComp
+Text Label 7500 2650 0    50   ~ 0
 5V
 $Comp
 L Custom:LT1818 U?
 U 1 1 5D1F178A
-P 7925 2900
-F 0 "U?" H 7950 2700 50  0000 L CNN
-F 1 "LT1818" H 7950 2775 50  0000 L CNN
-F 2 "" H 7925 2900 50  0001 C CNN
-F 3 "" H 7975 3100 50  0001 C CNN
-	1    7925 2900
+P 7600 2950
+F 0 "U?" H 7625 2750 50  0000 L CNN
+F 1 "LT1818" H 7625 2825 50  0000 L CNN
+F 2 "" H 7600 2950 50  0001 C CNN
+F 3 "" H 7650 3150 50  0001 C CNN
+	1    7600 2950
 	1    0    0    -1
 $EndComp
@@
 L Device:R R?
 U 1 1 5D1EC57B
-P 7475 2800
-F 0 "R?" V 7375 2850 50  0000 C CNN
-F 1 "R" V 7300 2875 50  0000 C CNN
-F 2 "" V 7405 2800 50  0001 C CNN
-F 3 "~" H 7475 2800 50  0001 C CNN
-	1    7475 2800
-	0    -1   -1   0
-$EndComp
-Wire Wire Line
-	7200 2800 7325 2800
-Wire Wire Line
-	7200 2500 7200 2800
+P 7200 2700
+F 0 "R?" H 7300 2775 50  0000 C CNN
+F 1 "R" H 7275 2700 50  0000 C CNN
+F 2 "" V 7130 2700 50  0001 C CNN
+F 3 "~" H 7200 2700 50  0001 C CNN
+	1    7200 2700
+	1    0    0    -1
+$EndComp
 $Comp
 L power:GNDA #PWR?
@@
 Wire Notes Line
 	4875 5900 4875 3675
-Text Label 8425 2900 0    50   ~ 0
+Text Label 8550 2950 0    50   ~ 0
 VID
 $Comp
@@
 	0    1    1    0
 $EndComp
+Text Label 10875 3450 0    50   ~ 0
+PHO2
+Wire Wire Line
+	10650 2150 10850 2150
+Wire Wire Line
+	10650 3350 10875 3350
+Wire Wire Line
+	10650 3150 10875 3150
+Text Label 10875 3350 0    50   ~ 0
+PHO3
+Text Label 10875 3150 0    50   ~ 0
+PHO4
+Wire Wire Line
+	7200 2500 7200 2550
+Wire Wire Line
+	7200 2850 7300 2850
+Wire Wire Line
+	7500 3250 7125 3250
+Wire Wire Line
+	7900 2950 8100 2950
+Wire Wire Line
+	7300 3050 7300 3350
+Wire Wire Line
+	7300 3350 7900 3350
+Wire Wire Line
+	7900 3350 7900 2950
+Connection ~ 7900 2950
+$Comp
+L Device:R R?
+U 1 1 5D369A7B
+P 8250 2950
+F 0 "R?" V 8043 2950 50  0000 C CNN
+F 1 "R" V 8134 2950 50  0000 C CNN
+F 2 "" V 8180 2950 50  0001 C CNN
+F 3 "~" H 8250 2950 50  0001 C CNN
+	1    8250 2950
+	0    1    1    0
+$EndComp
+$Comp
+L Device:C C?
+U 1 1 5D36AE0A
+P 8475 3100
+F 0 "C?" H 8250 3075 50  0000 L CNN
+F 1 "C" H 8250 3000 50  0000 L CNN
+F 2 "" H 8513 2950 50  0001 C CNN
+F 3 "~" H 8475 3100 50  0001 C CNN
+	1    8475 3100
+	1    0    0    -1
+$EndComp
+Wire Wire Line
+	8400 2950 8475 2950
+Connection ~ 8475 2950
+Wire Wire Line
+	8475 2950 8550 2950
+$Comp
+L Device:CP C?
+U 1 1 5D36F522
+P 6450 3300
+F 0 "C?" H 6650 3275 50  0000 R CNN
+F 1 "CP" H 6650 3350 50  0000 R CNN
+F 2 "" H 6488 3150 50  0001 C CNN
+F 3 "~" H 6450 3300 50  0001 C CNN
+	1    6450 3300
+	-1   0    0    1
+$EndComp
+Wire Notes Line
+	8700 3575 4875 3575
+$Comp
+L power:GNDA #PWR?
+U 1 1 5D37C278
+P 6800 3450
+F 0 "#PWR?" H 6800 3200 50  0001 C CNN
+F 1 "GNDA" H 6625 3375 50  0000 C CNN
+F 2 "" H 6800 3450 50  0001 C CNN
+F 3 "" H 6800 3450 50  0001 C CNN
+	1    6800 3450
+	1    0    0    -1
+$EndComp
+$Comp
+L Device:C C?
+U 1 1 5D3836C3
+P 6800 3300
+F 0 "C?" H 6600 3325 50  0000 L CNN
+F 1 "C" H 6600 3250 50  0000 L CNN
+F 2 "" H 6838 3150 50  0001 C CNN
+F 3 "~" H 6800 3300 50  0001 C CNN
+	1    6800 3300
+	1    0    0    -1
+$EndComp
+$Comp
+L power:-5V #PWR?
+U 1 1 5D3A19D2
+P 7125 3250
+F 0 "#PWR?" H 7125 3350 50  0001 C CNN
+F 1 "-5V" H 7140 3423 50  0000 C CNN
+F 2 "" H 7125 3250 50  0001 C CNN
+F 3 "" H 7125 3250 50  0001 C CNN
+	1    7125 3250
+	1    0    0    -1
+$EndComp
+Wire Wire Line
+	7125 3250 7025 3250
+Wire Wire Line
+	7025 3250 7025 3150
+Wire Wire Line
+	7025 3150 6800 3150
+Connection ~ 7125 3250
+Connection ~ 6800 3150
+Wire Wire Line
+	6800 3150 6450 3150
+Text Label 4200 4550 0    50   ~ 0
+TRIG
+Text Label 10875 3650 0    50   ~ 0
+B1
+Text Label 10875 3950 0    50   ~ 0
+B2
+Wire Wire Line
+	10650 3950 10875 3950
+Wire Wire Line
+	10650 4050 10875 4050
+Wire Wire Line
+	10650 4150 10875 4150
+Wire Wire Line
+	10650 4250 10875 4250
+Wire Wire Line
+	10650 4350 10875 4350
+Wire Wire Line
+	10650 4450 10875 4450
+Text Label 10875 4050 0    50   ~ 0
+B3
+Text Label 10875 4150 0    50   ~ 0
+B4
+Text Label 10875 4250 0    50   ~ 0
+B5
+Text Label 10875 4350 0    50   ~ 0
+B6
+Text Label 10875 4450 0    50   ~ 0
+B7
+Text Label 10875 3750 0    50   ~ 0
+B8
+Wire Wire Line
+	10650 3650 10875 3650
+Text Label 10875 2550 0    50   ~ 0
+B9
+Text Label 10875 2450 0    50   ~ 0
+B10
+Wire Wire Line
+	10650 2450 10875 2450
+Wire Wire Line
+	10650 2550 10875 2550
 $EndSCHEMATC

Commit message: sch review changes, eeprom, linear image sensor.
Parts:
- removed C? (x3): C_Small, symbol Device:C_Small
- removed C? (x2): CP1_Small, symbol Device:CP1_Small
- removed C? (x2): C, symbol Device:C
- removed C?: CP, symbol Device:CP
- removed R? (x6): R, symbol Device:R
- removed U?: ATmega32U4-MU, Package_DFN_QFN:QFN-44-1EP_7x7mm_P0.5mm_EP5.2x5.2mm, symbol MCU_Microchip_ATmega:ATmega32U4-MU
- removed U? (x4): S1336-44BQ, symbol Custom:S1336-44BQ
- removed U? (x4): OPAMP, symbol pspice:OPAMP
- removed U?: S14739-20, symbol Custom:S14739-20
- removed U?: LT1818, symbol Custom:LT1818
- removed U?: MCP9700AT-HLT, Package_TO_SOT_SMD:SOT-353_SC-70-5, symbol Sensor_Temperature:MCP9700AT-HLT
- added C? (x5): 0.1uF, symbol Device:C_Small
- added C?: 22pF, symbol Device:C_Small
- added C? (x5): 22uF, symbol Device:CP_Small
- added C? (x2): 1uF, symbol Device:C_Small
- added J?: Screw_Terminal_01x09, symbol Connector:Screw_Terminal_01x09
- added R? (x2): 82, symbol Device:R_Small
- added R?: 100, symbol Device:R_Small
- added R?: 51, symbol Device:R_Small
- added U?: S14739-20, symbol Custom:S14739-20
- added U?: LT1818, symbol Custom:LT1818
- added U?: 74HC541, symbol Custom:74HC541
- added U?: MCP9701A, symbol Custom:MCP9701A
Connections:
- net labels added: CLK, eos, trig
- net labels removed: 5V, B1, B10, B2, B3, B4, B5, B6, B7, B8, B9, PHO1, PHO2, PHO3, PHO4, SDA, SQW, Trig
- wire segments 103 -> 60
Other:
- note added: "BURT"
- note added: "CMOS Image Sensor\nMode: global shutter\nInput: 5V Vdd\nOutput: Digital VIDEO_S"
- note removed: "Microcontroller"
- note removed: "Photodiodes"
- note removed: "Spectrometer"
- moved on the sheet: D?, R?

Commit message: battery and burn wire circuitry, motor driver *incomplete
Parts:
- added C?: 4.7uF, symbol Device:C_Small
- added D? (x2): D, symbol Device:D
- added M?: Motor_DC, symbol Motor:Motor_DC
- added Q? (x5): Q_NMOS_DGS, symbol Device:Q_NMOS_DGS
- added R? (x2): R_Small, symbol Device:R_Small
- added R? (x5): BURNWIRE, symbol Device:R
- added R? (x5): 10k, symbol Device:R
- added U?: MCP73831-DFN, symbol Custom:MCP73831-DFN
- added U?: A3908, symbol Custom:A3908
Connections:
- net labels added: +BATT, B1, B2, B3, B4, B5, START_VID
- wire segments 60 -> 123
Other:
- note added: "OUTPUT\nOUTPUT\nINPUT\nINPUT\n"
- moved on the sheet: C?, J?, R?, U?

Commit message: motor driver
Parts:
- added R?: 18k, symbol Device:R_Small
- added R?: 10k, symbol Device:R_Small
Changed lines of the file:
@@
+	1    0    0    -1
+$EndComp
+$Comp
+L Device:R_Small R?
+U 1 1 5D538E55
+P -950 5475
+F 0 "R?" H -891 5521 50  0000 L CNN
+F 1 "18k" H -891 5430 50  0000 L CNN
+F 2 "" H -950 5475 50  0001 C CNN
+F 3 "~" H -950 5475 50  0001 C CNN
+	1    -950 5475
+	1    0    0    -1
+$EndComp
+$Comp
+L Device:R_Small R?
+U 1 1 5D543F60
+P -950 5775
+F 0 "R?" H -1100 5750 50  0000 L CNN
+F 1 "10k" H -1150 5675 50  0000 L CNN
+F 2 "" H -950 5775 50  0001 C CNN
+F 3 "~" H -950 5775 50  0001 C CNN
+	1    -950 5775
 	1    0    0    -1
 $EndComp

Commit message: burt for review
Parts:
- removed D?: D, symbol Device:D
- removed J?: Conn_02x03_Counter_Clockwise, symbol Connector_Generic:Conn_02x03_Counter_Clockwise
- added Q? (x5): Q_NMOS_DGS, symbol Device:Q_NMOS_DGS
- added R? (x5): BURNWIRE, symbol Device:R
- added R? (x5): 10k, symbol Device:R
Connections:
- net labels added: BL1, BL2, BL3, BL4, BL5, BL6, BL7, BL8, BP1, BP2, IN1, IN2
- net labels removed: MISO, MOSI, RST, SCK
- wire segments 123 -> 164
Other:
- note removed: "OUTPUT\nOUTPUT\nINPUT\nINPUT\n"
- note removed: "Programming Header"
- moved on the sheet: C?, D?, J?, M?, Q?, R?, U?

Commit message: Fixed symbol libraries
Parts:
- U?: symbol Custom:S14739-20 -> Burt-rescue:S14739-20-Custom
- U?: symbol Custom:LT1818 -> Burt-rescue:LT1818-Custom
- U?: symbol Custom:MCP73831-DFN -> Burt-rescue:MCP73831-DFN-Custom
- U?: symbol Custom:74HC541 -> Burt-rescue:74HC541-Custom
- U?: symbol Custom:MCP9701A -> Burt-rescue:MCP9701A-Custom
- U?: symbol Custom:A3908 -> Burt-rescue:A3908-Custom
Changed lines of the file:
@@
 $EndComp
 $Comp
-L Custom:LT1818 U?
+L Burt-rescue:LT1818-Custom U?
 U 1 1 5D25B2EA
 P 5425 2375
@@
 	4875 1375 4950 1375
 $Comp
-L Custom:74HC541 U?
+L Burt-rescue:74HC541-Custom U?
 U 1 1 5D287D5C
 P 2025 2025
@@
 START_VID
 $Comp
-L Custom:S14739-20 U?
+L Burt-rescue:S14739-20-Custom U?
 U 1 1 5D25536A
 P 4425 1525
@@
 Connection ~ 1600 6800
 $Comp
-L Custom:A3908 U?
+L Burt-rescue:A3908-Custom U?
 U 1 1 5D5325EF
 P 4450 6650
@@
 $EndComp
 $Comp
-L Custom:MCP73831-DFN U?
+L Burt-rescue:MCP73831-DFN-Custom U?
 U 1 1 5D264C9F
 P 2000 6600
@@
 $EndComp
 $Comp
-L Custom:MCP9701A U?
+L Burt-rescue:MCP9701A-Custom U?
 U 1 1 5D425D1D
 P 4775 4175
