File: Circuitry/Burt/Burt.sch (KiCad schematic (older format))
At the start: 67 parts

Commit message: Changed burt some
Parts:
- added BT?: Battery_Cell, symbol Device:Battery_Cell
- added C?: 4.7uF, symbol Device:C_Small
- J?: value Screw_Terminal_01x09 -> Screw_Terminal_01x011; symbol Connector:Screw_Terminal_01x09 -> Connector:Screw_Terminal_01x11
- R?: value R_Small -> 470R
- R?: value R_Small -> 20k
- R?: value 51 -> 51R
Connections:
- net +BATT: now also BT?.1 (+), C?.1
- net GND: now also BT?.2 (-), C?.2
- net IN1: now also J?.10 (Pin_10)
- net IN2: now also J?.11 (Pin_11)
Other:
- note added: "Charging and Battery"
- note added: "SET TO 50 mA"
- moved on the sheet: C?, D?, R?, U?
Changed lines of the file:
@@
 Text Notes 7000 6750 0    118  ~ 24
 BURT
+Text Label 5925 6450 2    50   ~ 0
+TEMP
 Text Label 5925 6550 2    50   ~ 0
-TEMP
+VID
 Text Label 5925 6650 2    50   ~ 0
-VID
-Text Label 5925 6750 2    50   ~ 0
 CRYSTAL
 $Comp
@@
 P 5975 2375
 F 0 "R?" V 5800 2500 50  0000 C CNN
-F 1 "51" V 5875 2500 50  0000 C CNN
+F 1 "51R" V 5875 2500 50  0000 C CNN
 F 2 "" H 5975 2375 50  0001 C CNN
 F 3 "~" H 5975 2375 50  0001 C CNN
@@
 CRYSTAL
 $Comp
-L Connector:Screw_Terminal_01x09 J?
+L Connector:Screw_Terminal_01x11 J?
 U 1 1 5D3FE5E4
 P 6125 6950
 F 0 "J?" H 5475 7550 50  0000 L CNN
-F 1 "Screw_Terminal_01x09" H 5475 7675 50  0000 L CNN
+F 1 "Screw_Terminal_01x011" H 5475 7675 50  0000 L CNN
 F 2 "" H 6125 6950 50  0001 C CNN
 F 3 "~" H 6125 6950 50  0001 C CNN
@@
 	1    0    0    -1
 $EndComp
-Text Label 5925 6850 2    50   ~ 0
+Text Label 5925 6750 2    50   ~ 0
 START_VID
 $Comp
@@
 L Device:R_Small R?
 U 1 1 5D28D225
-P 2400 7075
-F 0 "R?" H 2459 7121 50  0000 L CNN
-F 1 "R_Small" H 2459 7030 50  0000 L CNN
-F 2 "" H 2400 7075 50  0001 C CNN
-F 3 "~" H 2400 7075 50  0001 C CNN
-	1    2400 7075
+P 2750 5775
+F 0 "R?" H 2809 5821 50  0000 L CNN
+F 1 "470R" H 2809 5730 50  0000 L CNN
+F 2 "" H 2750 5775 50  0001 C CNN
+F 3 "~" H 2750 5775 50  0001 C CNN
+	1    2750 5775
 	1    0    0    -1
 $EndComp
@@
 L Device:R_Small R?
 U 1 1 5D28D9E9
-P 2575 6525
-F 0 "R?" H 2516 6479 50  0000 R CNN
-F 1 "R_Small" H 2516 6570 50  0000 R CNN
-F 2 "" H 2575 6525 50  0001 C CNN
-F 3 "~" H 2575 6525 50  0001 C CNN
-	1    2575 6525
+P 2925 5225
+F 0 "R?" H 2866 5179 50  0000 R CNN
+F 1 "20k" H 2866 5270 50  0000 R CNN
+F 2 "" H 2925 5225 50  0001 C CNN
+F 3 "~" H 2925 5225 50  0001 C CNN
+	1    2925 5225
 	-1   0    0    1
 $EndComp
 Wire Wire Line
-	2400 6300 2575 6300
-Wire Wire Line
-	2575 6300 2575 6425
-Wire Wire Line
-	2400 6700 2575 6700
-Wire Wire Line
-	2575 6700 2575 6625
+	2750 5000 2925 5000
+Wire Wire Line
+	2925 5000 2925 5125
+Wire Wire Line
+	2750 5400 2925 5400
+Wire Wire Line
+	2925 5400 2925 5325
 $Comp
 L power:GND #PWR?
 U 1 1 5D292366
-P 2575 6700
-F 0 "#PWR?" H 2575 6450 50  0001 C CNN
-F 1 "GND" H 2580 6527 50  0000 C CNN
-F 2 "" H 2575 6700 50  0001 C CNN
-F 3 "" H 2575 6700 50  0001 C CNN
-	1    2575 6700
-	1    0    0    -1
-$EndComp
-Connection ~ 2575 6700
+P 2925 5400
+F 0 "#PWR?" H 2925 5150 50  0001 C CNN
+F 1 "GND" H 2930 5227 50  0000 C CNN
+F 2 "" H 2925 5400 50  0001 C CNN
+F 3 "" H 2925 5400 50  0001 C CNN
+	1    2925 5400
+	1    0    0    -1
+$EndComp
+Connection ~ 2925 5400
 $Comp
 L Device:C_Small C?
 U 1 1 5D2929F0
-P 925 6400
-F 0 "C?" H 725 6425 50  0000 L CNN
-F 1 "4.7uF" H 600 6325 50  0000 L CNN
-F 2 "" H 925 6400 50  0001 C CNN
-F 3 "~" H 925 6400 50  0001 C CNN
-	1    925  6400
+P 1275 5100
+F 0 "C?" H 1075 5125 50  0000 L CNN
+F 1 "4.7uF" H 950 5025 50  0000 L CNN
+F 2 "" H 1275 5100 50  0001 C CNN
+F 3 "~" H 1275 5100 50  0001 C CNN
+	1    1275 5100
 	1    0    0    -1
 $EndComp
@@
 L Device:D D?
 U 1 1 5D29968B
-P 1150 6450
-F 0 "D?" V 1196 6371 50  0000 R CNN
-F 1 "D" V 1105 6371 50  0000 R CNN
-F 2 "" H 1150 6450 50  0001 C CNN
-F 3 "~" H 1150 6450 50  0001 C CNN
-	1    1150 6450
+P 1500 5150
+F 0 "D?" V 1546 5071 50  0000 R CNN
+F 1 "D" V 1455 5071 50  0000 R CNN
+F 2 "" H 1500 5150 50  0001 C CNN
+F 3 "~" H 1500 5150 50  0001 C CNN
+	1    1500 5150
 	0    -1   -1   0
 $EndComp
 Wire Wire Line
-	800  6300 925  6300
-Connection ~ 925  6300
-Wire Wire Line
-	925  6300 1150 6300
-Connection ~ 1150 6300
-Wire Wire Line
-	1150 6300 1425 6300
-Wire Wire Line
-	1425 6300 1425 6500
-Wire Wire Line
-	1425 6500 1600 6500
-Connection ~ 1425 6300
-Wire Wire Line
-	1425 6300 1600 6300
-Wire Wire Line
-	2400 6900 2400 6975
-Wire Wire Line
-	1150 6600 1150 7350
-Wire Wire Line
-	1150 7350 2400 7350
-Wire Wire Line
-	2400 7350 2400 7175
+	1150 5000 1275 5000
+Connection ~ 1275 5000
+Wire Wire Line
+	1275 5000 1500 5000
+Connection ~ 1500 5000
+Wire Wire Line
+	1500 5000 1775 5000
+Wire Wire Line
+	1775 5000 1775 5200
+Wire Wire Line
+	1775 5200 1950 5200
+Connection ~ 1775 5000
+Wire Wire Line
+	1775 5000 1950 5000
+Wire Wire Line
+	2750 5600 2750 5675
+Wire Wire Line
+	1500 5300 1500 6050
+Wire Wire Line
+	1500 6050 2750 6050
+Wire Wire Line
+	2750 6050 2750 5875
 $Comp
 L power:GND #PWR?
 U 1 1 5D2BE8A0
-P 925 6500
-F 0 "#PWR?" H 925 6250 50  0001 C CNN
-F 1 "GND" H 930 6327 50  0000 C CNN
-F 2 "" H 925 6500 50  0001 C CNN
-F 3 "" H 925 6500 50  0001 C CNN
-	1    925  6500
+P 1275 5200
+F 0 "#PWR?" H 1275 4950 50  0001 C CNN
+F 1 "GND" H 1280 5027 50  0000 C CNN
+F 2 "" H 1275 5200 50  0001 C CNN
+F 3 "" H 1275 5200 50  0001 C CNN
+	1    1275 5200
 	1    0    0    -1
 $EndComp
 Wire Notes Line
 	625  3250 6750 3250
+Text Label 5925 6850 2    50   ~ 0
+B1
 Text Label 5925 6950 2    50   ~ 0
-B1
+B2
+Text Label 5925 7250 2    50   ~ 0
+B5
+Text Label 5925 7150 2    50   ~ 0
+B4
 Text Label 5925 7050 2    50   ~ 0
-B2
-Text Label 5925 7350 2    50   ~ 0
-B5
-Text Label 5925 7250 2    50   ~ 0
-B4
-Text Label 5925 7150 2    50   ~ 0
 B3
 $Comp
@@
 L power:+BATT #PWR?
 U 1 1 5D46466E
-P 1300 6800
-F 0 "#PWR?" H 1300 6650 50  0001 C CNN
-F 1 "+BATT" H 1315 6973 50  0000 C CNN
-F 2 "" H 1300 6800 50  0001 C CNN
-F 3 "" H 1300 6800 50  0001 C CNN
-	1    1300 6800
-	1    0    0    -1
-$EndComp
-Wire Wire Line
-	1600 6700 1600 6800
-Wire Wire Line
-	1600 6800 1300 6800
-Wire Wire Line
-	1600 6900 1600 6800
-Connection ~ 1600 6800
+P 1650 5500
+F 0 "#PWR?" H 1650 5350 50  0001 C CNN
+F 1 "+BATT" H 1665 5673 50  0000 C CNN
+F 2 "" H 1650 5500 50  0001 C CNN
+F 3 "" H 1650 5500 50  0001 C CNN
+	1    1650 5500
+	1    0    0    -1
+$EndComp
+Wire Wire Line
+	1950 5400 1950 5500
+Wire Wire Line
+	1950 5500 1825 5500
+Wire Wire Line
+	1950 5600 1950 5500
+Connection ~ 1950 5500
 $Comp
 L Burt-rescue:A3908-Custom U?
@@
 L power:+5V #PWR?
 U 1 1 5D287139
-P 800 6300
-F 0 "#PWR?" H 800 6150 50  0001 C CNN
-F 1 "+5V" H 815 6473 50  0000 C CNN
-F 2 "" H 800 6300 50  0001 C CNN
-F 3 "" H 800 6300 50  0001 C CNN
-	1    800  6300
+P 1150 5000
+F 0 "#PWR?" H 1150 4850 50  0001 C CNN
+F 1 "+5V" H 1165 5173 50  0000 C CNN
+F 2 "" H 1150 5000 50  0001 C CNN
+F 3 "" H 1150 5000 50  0001 C CNN
+	1    1150 5000
 	1    0    0    -1
 $EndComp
@@
 L Burt-rescue:MCP73831-DFN-Custom U?
 U 1 1 5D264C9F
-P 2000 6600
-F 0 "U?" H 2000 7215 50  0000 C CNN
-F 1 "MCP73831-DFN" H 2000 7124 50  0000 C CNN
-F 2 "" H 2000 6600 50  0001 C CNN
-F 3 "" H 2000 6600 50  0001 C CNN
-	1    2000 6600
+P 2350 5300
+F 0 "U?" H 2350 5915 50  0000 C CNN
+F 1 "MCP73831-DFN" H 2350 5824 50  0000 C CNN
+F 2 "" H 2350 5300 50  0001 C CNN
+F 3 "" H 2350 5300 50  0001 C CNN
+	1    2350 5300
 	1    0    0    -1
 $EndComp
@@
 Wire Notes Line
 	6750 4825 5475 4825
+Text Label 5925 7350 2    50   ~ 0
+IN1
+Text Label 5925 7450 2    50   ~ 0
+IN2
+$Comp
+L Device:C_Small C?
+U 1 1 5D28C167
+P 1825 5600
+F 0 "C?" H 1625 5625 50  0000 L CNN
+F 1 "4.7uF" H 1500 5525 50  0000 L CNN
+F 2 "" H 1825 5600 50  0001 C CNN
+F 3 "~" H 1825 5600 50  0001 C CNN
+	1    1825 5600
+	1    0    0    -1
+$EndComp
+Connection ~ 1825 5500
+Wire Wire Line
+	1825 5500 1650 5500
+$Comp
+L power:GND #PWR?
+U 1 1 5D28CAB7
+P 1825 5700
+F 0 "#PWR?" H 1825 5450 50  0001 C CNN
+F 1 "GND" H 1830 5527 50  0000 C CNN
+F 2 "" H 1825 5700 50  0001 C CNN
+F 3 "" H 1825 5700 50  0001 C CNN
+	1    1825 5700
+	1    0    0    -1
+$EndComp
+Text Notes 3125 5225 0    50   ~ 0
+SET TO 50 mA
+$Comp
+L Device:Battery_Cell BT?
+U 1 1 5D28E83B
+P 925 5700
+F 0 "BT?" H 1043 5796 50  0000 L CNN
+F 1 "Battery_Cell" H 1043 5705 50  0000 L CNN
+F 2 "" V 925 5760 50  0001 C CNN
+F 3 "~" V 925 5760 50  0001 C CNN
+	1    925  5700
+	1    0    0    -1
+$EndComp
+$Comp
+L power:+BATT #PWR?
+U 1 1 5D291146
+P 925 5500
+F 0 "#PWR?" H 925 5350 50  0001 C CNN
+F 1 "+BATT" H 940 5673 50  0000 C CNN
+F 2 "" H 925 5500 50  0001 C CNN
+F 3 "" H 925 5500 50  0001 C CNN
+	1    925  5500
+	1    0    0    -1
+$EndComp
+$Comp
+L power:GND #PWR?
+U 1 1 5D291472
+P 925 5800
+F 0 "#PWR?" H 925 5550 50  0001 C CNN
+F 1 "GND" H 930 5627 50  0000 C CNN
+F 2 "" H 925 5800 50  0001 C CNN
+F 3 "" H 925 5800 50  0001 C CNN
+	1    925  5800
+	1    0    0    -1
+$EndComp
+Wire Notes Line
+	825  4575 3675 4575
+Wire Notes Line
+	3675 4575 3675 6175
+Wire Notes Line
+	3675 6175 825  6175
+Wire Notes Line
+	825  6175 825  4575
+Text Notes 825  4675 0    50   ~ 0
+Charging and Battery
 $EndSCHEMATC
