File: Circuitry/Burt/Burt.sch (KiCad schematic (older format))
At the start: 40 parts, among them J1 Conn_01x17, J2 Conn_01x08_Female, M1 Motor_DC, Q1 SSM6N58NU, Q2 SSM6N58NU, Q3 SSM6N58NU, Q4 SSM6N58NU, Q5 SSM6N58NU, U1 MCP9701A, U2 A3908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

Commit message: Made a new ribbon cable connector
Parts:
- removed J1: Conn_01x17, Custom:0522071733, symbol Connector_Generic:Conn_01x17
- added J1: Conn_01x20, Custom:62674-201121ALF, symbol Connector_Generic:Conn_01x20
- J2: footprint Connector_PinHeader_2.54mm:PinHeader_1x08_P2.54mm_Vertical -> Connector_PinHeader_2.54mm:PinHeader_1x08_P2.54mm_Horizontal
Connections:
- net CS is gone; now on net CS_IMG: J2.1 (Pin_1)
- net +3V3: now also J1.15 (Pin_15)
- net +5V: now also J1.16 (Pin_16)
- net +BATT: now also BT1.1 (+), C2.1, U3.3 (Vbat)
- net BL1: now also Q1.2 (G), R8.2; no longer Q2.2 (G), Q3.5 (G), R1.2, R9.2
- net BL2: now also Q1.5 (G), R18.2; no longer Q2.5 (G), Q4.2 (G), R10.2, R2.2
- net BL3: now also Q2.2 (G), R1.2
- net BL4: now also Q2.5 (G), R2.2
- net BL5: now also Q3.2 (G), R3.2; no longer Q1.2 (G), Q5.2 (G), R19.2, R8.2
- net BL6: now also Q3.5 (G), R9.2; no longer Q4.5 (G), Q5.5 (G), R17.2, R20.2
- net BL7: now also Q4.2 (G), R10.2
- net BL8: now also Q4.5 (G), R17.2
- net BP1: now also Q5.2 (G), R19.2, J1.8 (Pin_8); no longer Q3.2 (G), R3.2
- net BP2: now also Q5.5 (G), R20.2, J1.9 (Pin_9); no longer Q1.5 (G), R18.2
- net CS_IMG: now also J1.2 (Pin_2)
- net GND: now also J1.17 (Pin_17)
- net IN1: now also J1.13 (Pin_13)
- net IN2: now also J1.14 (Pin_14)
- net MISO: now also J1.4 (Pin_4)
- net MOSI: now also J1.3 (Pin_3)
- net RCLK: now also J1.12 (Pin_12)
- net SCK: now also J1.5 (Pin_5)
- net SCL: now also J1.7 (Pin_7)
- net SDA: now also J1.6 (Pin_6)
- net SER: now also J1.10 (Pin_10)
- net SRCLK: now also J1.11 (Pin_11)
- net TEMP: now also J1.1 (Pin_1)
- no-connect marks 1 -> 4
Other:
- moved on the sheet: Q1A, Q1B, Q2A, Q2B, Q3A, Q3B, Q4B, Q5A, Q5B, R1, R11, R12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
