File: Circuitry/Joe/Joe.sch (KiCad schematic (older format))
At the start: 32 parts, among them J1 Conn_02x03_Counter_Clockwise, J2 Conn_01x17, J3 USB_B_Micro, J4 Micro_SD_Card, U5 DS3231MZ, U6 M24C32-XDW5TP, U7 DF12-20DS, U8 AP2127N-3.3, U9 ATmega32U4-MU

Commit message: joe footprints, symbols, and sch reviewed
Connections:
- wire segments 102 -> 101
- no-connect marks 16 -> 17
Changed lines of the file:
@@
 L power:+3V3 #PWR036
 U 1 1 5D38F4D1
-P 10400 1150
-F 0 "#PWR036" H 10400 1000 50  0001 C CNN
-F 1 "+3V3" H 10415 1323 50  0000 C CNN
-F 2 "" H 10400 1150 50  0001 C CNN
-F 3 "" H 10400 1150 50  0001 C CNN
-	1    10400 1150
-	1    0    0    -1
-$EndComp
-Wire Wire Line
-	10400 1150 10325 1150
+P 10325 1150
+F 0 "#PWR036" H 10325 1000 50  0001 C CNN
+F 1 "+3V3" H 10340 1323 50  0000 C CNN
+F 2 "" H 10325 1150 50  0001 C CNN
+F 3 "" H 10325 1150 50  0001 C CNN
+	1    10325 1150
+	1    0    0    -1
+$EndComp
 NoConn ~ 7425 3200
 $Comp
@@
 	1    0    0    -1
 $EndComp
+NoConn ~ 10625 5050
 $EndSCHEMATC

Commit message: joe layout
Parts:
- removed J2: Conn_01x17, Custom:0522071733, symbol Connector_Generic:Conn_01x17
- added J2: Conn_01x20, Custom:62674-201121ALF, symbol Connector_Generic:Conn_01x20
Connections:
- wire segments 101 -> 105
- no-connect marks 17 -> 22
Changed lines of the file:
@@
 Text Label 9225 2650 2    50   ~ 0
 RST
-Text Label 10825 3350 0    50   ~ 0
+Text Label 10850 4350 0    50   ~ 0
 TMR_RST
 Wire Wire Line
@@
 Wire Wire Line
 	3075 6325 2900 6325
-Text Label 10850 5350 0    50   ~ 0
+Text Label 10825 3350 0    50   ~ 0
 WC
 Wire Notes Line
@@
 L power:+3V3 #PWR037
 U 1 1 5D47F25B
-P 4775 4325
-F 0 "#PWR037" H 4775 4175 50  0001 C CNN
-F 1 "+3V3" V 4790 4453 50  0000 L CNN
-F 2 "" H 4775 4325 50  0001 C CNN
-F 3 "" H 4775 4325 50  0001 C CNN
-	1    4775 4325
+P 4650 4325
+F 0 "#PWR037" H 4650 4175 50  0001 C CNN
+F 1 "+3V3" V 4665 4453 50  0000 L CNN
+F 2 "" H 4650 4325 50  0001 C CNN
+F 3 "" H 4650 4325 50  0001 C CNN
+	1    4650 4325
 	0    -1   -1   0
 $EndComp
@@
 L power:+5V #PWR038
 U 1 1 5D480338
-P 4775 4425
-F 0 "#PWR038" H 4775 4275 50  0001 C CNN
-F 1 "+5V" V 4790 4553 50  0000 L CNN
-F 2 "" H 4775 4425 50  0001 C CNN
-F 3 "" H 4775 4425 50  0001 C CNN
-	1    4775 4425
+P 4650 4425
+F 0 "#PWR038" H 4650 4275 50  0001 C CNN
+F 1 "+5V" V 4665 4553 50  0000 L CNN
+F 2 "" H 4650 4425 50  0001 C CNN
+F 3 "" H 4650 4425 50  0001 C CNN
+	1    4650 4425
 	0    -1   -1   0
 $EndComp
@@
 L power:GND #PWR039
 U 1 1 5D480BD6
-P 4775 4525
-F 0 "#PWR039" H 4775 4275 50  0001 C CNN
-F 1 "GND" H 4780 4352 50  0000 C CNN
-F 2 "" H 4775 4525 50  0001 C CNN
-F 3 "" H 4775 4525 50  0001 C CNN
-	1    4775 4525
-	1    0    0    -1
-$EndComp
-Text Label 10625 4350 0    50   ~ 0
+P 4600 4525
+F 0 "#PWR039" H 4600 4275 50  0001 C CNN
+F 1 "GND" H 4605 4352 50  0000 C CNN
+F 2 "" H 4600 4525 50  0001 C CNN
+F 3 "" H 4600 4525 50  0001 C CNN
+	1    4600 4525
+	1    0    0    -1
+$EndComp
+Text Label 10850 5350 0    50   ~ 0
 BUSY
 NoConn ~ 4450 1375
-$Comp
-L Connector_Generic:Conn_01x17 J2
-U 1 1 5D48D629
-P 4975 3725
-F 0 "J2" V 5075 3600 50  0000 L CNN
-F 1 "Conn_01x17" V 5075 3825 50  0000 L CNN
-F 2 "Custom:0522071733" H 4975 3725 50  0001 C CNN
-F 3 "~" H 4975 3725 50  0001 C CNN
-F 4 "https://www.digikey.com/product-detail/en/molex/0522071733/WM10952CT-ND/5170967" H 4975 3725 50  0001 C CNN "Part URL"
-	1    4975 3725
-	1    0    0    -1
-$EndComp
-Wire Notes Line
-	4200 4775 6200 4775
 $Comp
 L Joe-rescue:UFDFPN8-MC-Custom U6
@@
 $EndComp
 NoConn ~ 10625 5050
+$Comp
+L Connector_Generic:Conn_01x20 J2
+U 1 1 5D2D5DCB
+P 4975 3825
+F 0 "J2" H 5055 3817 50  0000 L CNN
+F 1 "Conn_01x20" H 5055 3726 50  0000 L CNN
+F 2 "Custom:62674-201121ALF" H 4975 3825 50  0001 C CNN
+F 3 "~" H 4975 3825 50  0001 C CNN
+	1    4975 3825
+	1    0    0    -1
+$EndComp
+Wire Wire Line
+	4650 4325 4775 4325
+Wire Wire Line
+	4650 4425 4775 4425
+Wire Wire Line
+	4600 4525 4775 4525
+NoConn ~ 4775 4625
+NoConn ~ 4775 4725
+NoConn ~ 4775 4825
+NoConn ~ 5375 2825
+NoConn ~ 3200 5400
+Wire Wire Line
+	10625 4350 10850 4350
 $EndSCHEMATC

Commit message: completed joe layout for review; addresses for dcf
Parts:
- removed D2: LED, LED_SMD:LED_0603_1608Metric, symbol Device:LED
- removed R10: 440R, Resistor_SMD:R_0603_1608Metric, symbol Device:R
- R12, R13, R14, R15: footprint OptoDevice:R_LDR_10x8.5mm_P7.6mm_Vertical -> Connector_PinHeader_1.00mm:PinHeader_1x02_P1.00mm_Vertical
Connections:
- net PLED2 is gone; now on net TEMP: U9.33 (~HWB~/PE2)
- net BUSY: now also U9.29 (PB5); no longer U9.38 (PF5)
- net CS_IMG: now also U9.32 (PC7)
- net IN1: now also U9.38 (PF5)
- net IN2: now also U9.37 (PF6)
- net PHO1: now also U9.36 (PF7); no longer U9.28 (PB4)
- net PLED3: now also U9.28 (PB4); no longer U9.36 (PF7)
- net SER: now also U9.30 (PB6); no longer U9.37 (PF6)
- net TMR_RST: now also U9.12 (PB7); no longer U9.22 (PD5)
- net WC: now also U9.22 (PD5); no longer U9.12 (PB7)
- net ~CS_SD: now also U9.41 (PF0); no longer U9.32 (PC7)
- net BP1: no longer names the net of J2.8 (Pin_8)
- net BP1: no longer U9.29 (PB5)
- net BP2: no longer names the net of J2.9 (Pin_9)
- net BP2: no longer U9.30 (PB6)
- no-connect marks 22 -> 20
Other:
- moved on the sheet: D3, R11
Changed lines of the file:
@@
 	10625 4550 10850 4550
 Connection ~ 1150 1150
-Text Label 10825 3050 0    50   ~ 0
+Text Label 10850 5550 0    50   ~ 0
 PHO1
 Wire Wire Line
@@
 $EndComp
 $Comp
-L Device:LED D2
-U 1 1 5D19383C
-P 3475 4650
-F 0 "D2" H 3468 4866 50  0000 C CNN
-F 1 "LED" H 3468 4775 50  0000 C CNN
-F 2 "LED_SMD:LED_0603_1608Metric" H 3475 4650 50  0001 C CNN
-F 3 "~" H 3475 4650 50  0001 C CNN
-F 4 "https://www.digikey.com/product-detail/en/lite-on-inc/LTST-C191KRKT/160-1447-1-ND/386836" H 3475 4650 50  0001 C CNN "Part URL"
-	1    3475 4650
-	1    0    0    -1
-$EndComp
-$Comp
-L Device:R R10
-U 1 1 5D193842
-P 3175 4650
-F 0 "R10" V 2968 4650 50  0000 C CNN
-F 1 "440R" V 3059 4650 50  0000 C CNN
-F 2 "Resistor_SMD:R_0603_1608Metric" V 3105 4650 50  0001 C CNN
-F 3 "~" H 3175 4650 50  0001 C CNN
-F 4 "https://www.digikey.com/product-detail/en/yageo/RC0603FR-07442RL/311-442HRCT-ND/730189" H 3175 4650 50  0001 C CNN "Part URL"
-	1    3175 4650
-	0    1    1    0
-$EndComp
-$Comp
 L Device:LED D3
 U 1 1 5D195D15
-P 3475 4975
-F 0 "D3" H 3468 5191 50  0000 C CNN
-F 1 "LED" H 3468 5100 50  0000 C CNN
-F 2 "LED_SMD:LED_0603_1608Metric" H 3475 4975 50  0001 C CNN
-F 3 "~" H 3475 4975 50  0001 C CNN
-F 4 "https://www.digikey.com/product-detail/en/lite-on-inc/LTST-C191TBKT/160-1647-1-ND/573587" H 3475 4975 50  0001 C CNN "Part URL"
-	1    3475 4975
+P 3475 4750
+F 0 "D3" H 3468 4966 50  0000 C CNN
+F 1 "LED" H 3468 4875 50  0000 C CNN
+F 2 "LED_SMD:LED_0603_1608Metric" H 3475 4750 50  0001 C CNN
+F 3 "~" H 3475 4750 50  0001 C CNN
+F 4 "https://www.digikey.com/product-detail/en/lite-on-inc/LTST-C191TBKT/160-1647-1-ND/573587" H 3475 4750 50  0001 C CNN "Part URL"
+	1    3475 4750
 	1    0    0    -1
 $EndComp
@@
 L Device:R R11
 U 1 1 5D195D1B
-P 3175 4975
-F 0 "R11" V 2968 4975 50  0000 C CNN
-F 1 "440R" V 3059 4975 50  0000 C CNN
-F 2 "Resistor_SMD:R_0603_1608Metric" V 3105 4975 50  0001 C CNN
-F 3 "~" H 3175 4975 50  0001 C CNN
-F 4 "https://www.digikey.com/product-detail/en/yageo/RC0603FR-07442RL/311-442HRCT-ND/730189" H 3175 4975 50  0001 C CNN "Part URL"
-	1    3175 4975
+P 3175 4750
+F 0 "R11" V 2968 4750 50  0000 C CNN
+F 1 "440R" V 3059 4750 50  0000 C CNN
+F 2 "Resistor_SMD:R_0603_1608Metric" V 3105 4750 50  0001 C CNN
+F 3 "~" H 3175 4750 50  0001 C CNN
+F 4 "https://www.digikey.com/product-detail/en/yageo/RC0603FR-07442RL/311-442HRCT-ND/730189" H 3175 4750 50  0001 C CNN "Part URL"
+	1    3175 4750
 	0    1    1    0
 $EndComp
@@
 	2825 4325 3025 4325
 $Comp
-L power:GND #PWR015
-U 1 1 5D19BB8C
-P 2825 4650
-F 0 "#PWR015" H 2825 4400 50  0001 C CNN
-F 1 "GND" H 2830 4477 50  0000 C CNN
-F 2 "" H 2825 4650 50  0001 C CNN
-F 3 "" H 2825 4650 50  0001 C CNN
-	1    2825 4650
-	1    0    0    -1
-$EndComp
-Wire Wire Line
-	2825 4650 3025 4650
-$Comp
 L power:GND #PWR016
 U 1 1 5D19E020
-P 2825 4975
-F 0 "#PWR016" H 2825 4725 50  0001 C CNN
-F 1 "GND" H 2830 4802 50  0000 C CNN
-F 2 "" H 2825 4975 50  0001 C CNN
-F 3 "" H 2825 4975 50  0001 C CNN
-	1    2825 4975
-	1    0    0    -1
-$EndComp
-Wire Wire Line
-	2825 4975 3025 4975
+P 2825 4750
+F 0 "#PWR016" H 2825 4500 50  0001 C CNN
+F 1 "GND" H 2830 4577 50  0000 C CNN
+F 2 "" H 2825 4750 50  0001 C CNN
+F 3 "" H 2825 4750 50  0001 C CNN
+	1    2825 4750
+	1    0    0    -1
+$EndComp
+Wire Wire Line
+	2825 4750 3025 4750
 Text Label 5650 1375 0    50   ~ 0
 BUSY
@@
 Text Label 9225 2650 2    50   ~ 0
 RST
-Text Label 10850 4350 0    50   ~ 0
+Text Label 10825 3350 0    50   ~ 0
 TMR_RST
 Wire Wire Line
@@
 Wire Wire Line
 	3075 6325 2900 6325
-Text Label 10825 3350 0    50   ~ 0
+Text Label 10850 4350 0    50   ~ 0
 WC
 Wire Notes Line
@@
 Wire Notes Line
 	2650 3825 2650 2475
-Text Label 10850 5450 0    50   ~ 0
-SER
-Text Label 10825 3150 0    50   ~ 0
-BP1
-Text Label 10825 3250 0    50   ~ 0
-BP2
 Wire Notes Line
 	2650 3875 4150 3875
@@
 Wire Notes Line
 	6200 500  4050 500
-Text Label 4775 3625 2    50   ~ 0
-BP1
-Text Label 4775 3725 2    50   ~ 0
-BP2
 $Comp
 L Connector:Micro_SD_Card J4
@@
 NoConn ~ 6800 1900
 NoConn ~ 6800 1200
-Text Label 10850 3650 0    50   ~ 0
+Text Label 10850 5050 0    50   ~ 0
 ~CS_SD
 Wire Wire Line
@@
 	10625 2650 10825 2650
 Text Label 10850 4750 0    50   ~ 0
-PLED2
+TEMP
 Wire Wire Line
 	10625 4750 10850 4750
-Text Label 10850 5550 0    50   ~ 0
+Text Label 10825 3050 0    50   ~ 0
 PLED3
 Wire Wire Line
 	10625 5550 10850 5550
-Text Label 3625 4975 0    50   ~ 0
+Text Label 3625 4750 0    50   ~ 0
 PLED3
-Text Label 3625 4650 0    50   ~ 0
-PLED2
 Text Label 3625 4325 0    50   ~ 0
 PLED1
@@
 F 0 "R12" V 1325 3525 50  0000 C CNN
 F 1 "R_PHOTO" V 1416 3525 50  0000 C CNN
-F 2 "OptoDevice:R_LDR_10x8.5mm_P7.6mm_Vertical" V 1700 3275 50  0001 L CNN
+F 2 "Connector_PinHeader_1.00mm:PinHeader_1x02_P1.00mm_Vertical" V 1700 3275 50  0001 L CNN
 F 3 "~" H 1650 3475 50  0001 C CNN
 F 4 "https://www.digikey.com/product-detail/en/advanced-photonix/NSL-5910/NSL-5910-ND/5436028" H 1650 3525 50  0001 C CNN "Part URL"
@@
 F 0 "R13" V 1375 4650 50  0000 C CNN
 F 1 "R_PHOTO" V 1466 4650 50  0000 C CNN
-F 2 "OptoDevice:R_LDR_10x8.5mm_P7.6mm_Vertical" V 1750 4400 50  0001 L CNN
+F 2 "Connector_PinHeader_1.00mm:PinHeader_1x02_P1.00mm_Vertical" V 1750 4400 50  0001 L CNN
 F 3 "~" H 1700 4600 50  0001 C CNN
 F 4 "https://www.digikey.com/product-detail/en/advanced-photonix/NSL-5910/NSL-5910-ND/5436028" H 1700 4650 50  0001 C CNN "Part URL"
@@
 F 0 "R14" V 1400 5800 50  0000 C CNN
 F 1 "R_PHOTO" V 1491 5800 50  0000 C CNN
-F 2 "OptoDevice:R_LDR_10x8.5mm_P7.6mm_Vertical" V 1775 5550 50  0001 L CNN
+F 2 "Connector_PinHeader_1.00mm:PinHeader_1x02_P1.00mm_Vertical" V 1775 5550 50  0001 L CNN
 F 3 "~" H 1725 5750 50  0001 C CNN
 F 4 "https://www.digikey.com/product-detail/en/advanced-photonix/NSL-5910/NSL-5910-ND/5436028" H 1725 5800 50  0001 C CNN "Part URL"
@@
 F 0 "R15" V 1425 6950 50  0000 C CNN
 F 1 "R_PHOTO" V 1516 6950 50  0000 C CNN
-F 2 "OptoDevice:R_LDR_10x8.5mm_P7.6mm_Vertical" V 1800 6700 50  0001 L CNN
+F 2 "Connector_PinHeader_1.00mm:PinHeader_1x02_P1.00mm_Vertical" V 1800 6700 50  0001 L CNN
 F 3 "~" H 1750 6900 50  0001 C CNN
 F 4 "https://www.digikey.com/product-detail/en/advanced-photonix/NSL-5910/NSL-5910-ND/5436028" H 1750 6950 50  0001 C CNN "Part URL"
@@
 	1    0    0    -1
 $EndComp
-Text Label 10850 5350 0    50   ~ 0
-BUSY
 NoConn ~ 4450 1375
 $Comp
@@
 	1    0    0    -1
 $EndComp
-NoConn ~ 10625 5050
 $Comp
 L Connector_Generic:Conn_01x20 J2
@@
 NoConn ~ 4775 4725
 NoConn ~ 4775 4825
-NoConn ~ 5375 2825
 NoConn ~ 3200 5400
 Wire Wire Line
 	10625 4350 10850 4350
+Wire Wire Line
+	10625 5050 10850 5050
+Text Label 10850 3650 0    50   ~ 0
+CS_IMG
+Text Label 10825 3250 0    50   ~ 0
+SER
+Text Label 10825 3150 0    50   ~ 0
+BUSY
+Text Label 10850 5350 0    50   ~ 0
+IN1
+Text Label 10850 5450 0    50   ~ 0
+IN2
 $EndSCHEMATC

Commit message: complete joe layoutgit add .git add .git add . woooohooooooo!
Parts:
- R12, R13, R14, R15: footprint Connector_PinHeader_1.00mm:PinHeader_1x02_P1.00mm_Vertical -> Custom:PinHeader_1x02_P1.00mm_Vertical
Connections:
- net +3V3: now also J1.2 (Pin_2); no longer J1.6 (Pin_6)
- net GND: now also J1.6 (Pin_6); no longer J1.4 (Pin_4)
- net MOSI: now also J1.4 (Pin_4); no longer J1.5 (Pin_5)
- net PHO1: now also U9.26 (PD6); no longer U9.36 (PF7)
- net PHO2: now also U9.36 (PF7); no longer U9.27 (PD7)
- net PHO3: now also U9.8 (PB0); no longer U9.26 (PD6)
- net PLED1: now also U9.27 (PD7); no longer U9.8 (PB0)
- net RST: now also J1.5 (Pin_5); no longer J1.3 (Pin_3)
- net RX: now also U7.12 (TX), U9.21 (PD3); no longer U7.11 (RX), U9.20 (PD2)
- net SCK: now also J1.3 (Pin_3); no longer J1.2 (Pin_2)
- net TX: now also U7.11 (RX), U9.20 (PD2); no longer U7.12 (TX), U9.21 (PD3)
- no-connect marks 20 -> 19
Changed lines of the file:
@@
 Wire Wire Line
 	10125 2350 10025 2350
+Text Label 5650 1475 0    50   ~ 0
+TX
 Text Label 4450 1475 2    50   ~ 0
-TX
-Text Label 5650 1475 0    50   ~ 0
 RX
 $Comp
@@
 Text Label 2950 3150 2    50   ~ 0
 MISO
-Text Label 2950 3250 2    50   ~ 0
+Text Label 2950 3350 2    50   ~ 0
 SCK
-Text Label 2950 3350 2    50   ~ 0
+Text Label 3850 3250 0    50   ~ 0
 RST
 Wire Wire Line
-	3850 3150 3850 3075
-Text Label 3850 3250 0    50   ~ 0
+	2725 3250 2725 3175
+Text Label 3850 3350 0    50   ~ 0
 MOSI
 $Comp
 L power:GND #PWR020
 U 1 1 5D212296
-P 3850 3450
-F 0 "#PWR020" H 3850 3200 50  0001 C CNN
-F 1 "GND" H 3855 3277 50  0000 C CNN
-F 2 "" H 3850 3450 50  0001 C CNN
-F 3 "" H 3850 3450 50  0001 C CNN
-	1    3850 3450
+P 4050 3250
+F 0 "#PWR020" H 4050 3000 50  0001 C CNN
+F 1 "GND" H 4055 3077 50  0000 C CNN
+F 2 "" H 4050 3250 50  0001 C CNN
+F 3 "" H 4050 3250 50  0001 C CNN
+	1    4050 3250
 	1    0    0    -1
 $EndComp
@@
 TMR_RST
 Wire Wire Line
-	3650 3150 3850 3150
-Wire Wire Line
 	3650 3250 3850 3250
 Wire Wire Line
-	3650 3350 3850 3350
-Wire Wire Line
-	3850 3350 3850 3450
+	4050 3150 4050 3250
 Wire Wire Line
 	3150 3150 2950 3150
-Wire Wire Line
-	3150 3250 2950 3250
 Wire Wire Line
 	3150 3350 2950 3350
@@
 	10625 4550 10850 4550
 Connection ~ 1150 1150
-Text Label 10850 5550 0    50   ~ 0
+Text Label 10850 4450 0    50   ~ 0
 PHO1
 Wire Wire Line
@@
 Wire Wire Line
 	10625 4250 10850 4250
-Text Label 10850 4550 0    50   ~ 0
+Text Label 10850 5550 0    50   ~ 0
 PHO2
-Text Label 10850 4450 0    50   ~ 0
+Text Label 10825 2650 0    50   ~ 0
 PHO3
 Text Label 10850 4250 0    50   ~ 0
@@
 Wire Wire Line
 	8950 3950 9425 3950
+Text Label 10850 4150 0    50   ~ 0
+RX
 Text Label 10850 4050 0    50   ~ 0
-RX
-Text Label 10850 4150 0    50   ~ 0
 TX
 Wire Wire Line
@@
 L power:+3V3 #PWR019
 U 1 1 5D37B22F
-P 3850 3075
-F 0 "#PWR019" H 3850 2925 50  0001 C CNN
-F 1 "+3V3" H 3865 3248 50  0000 C CNN
-F 2 "" H 3850 3075 50  0001 C CNN
-F 3 "" H 3850 3075 50  0001 C CNN
-	1    3850 3075
+P 2725 3175
+F 0 "#PWR019" H 2725 3025 50  0001 C CNN
+F 1 "+3V3" H 2740 3348 50  0000 C CNN
+F 2 "" H 2725 3175 50  0001 C CNN
+F 3 "" H 2725 3175 50  0001 C CNN
+	1    2725 3175
 	1    0    0    -1
 $EndComp
@@
 Wire Notes Line
 	6275 3825 6275 500
-Text Label 10825 2650 0    50   ~ 0
+Text Label 10850 4550 0    50   ~ 0
 PLED1
 Wire Wire Line
@@
 F 0 "R12" V 1325 3525 50  0000 C CNN
 F 1 "R_PHOTO" V 1416 3525 50  0000 C CNN
-F 2 "Connector_PinHeader_1.00mm:PinHeader_1x02_P1.00mm_Vertical" V 1700 3275 50  0001 L CNN
+F 2 "Custom:PinHeader_1x02_P1.00mm_Vertical" V 1700 3275 50  0001 L CNN
 F 3 "~" H 1650 3475 50  0001 C CNN
 F 4 "https://www.digikey.com/product-detail/en/advanced-photonix/NSL-5910/NSL-5910-ND/5436028" H 1650 3525 50  0001 C CNN "Part URL"
@@
 F 0 "R13" V 1375 4650 50  0000 C CNN
 F 1 "R_PHOTO" V 1466 4650 50  0000 C CNN
-F 2 "Connector_PinHeader_1.00mm:PinHeader_1x02_P1.00mm_Vertical" V 1750 4400 50  0001 L CNN
+F 2 "Custom:PinHeader_1x02_P1.00mm_Vertical" V 1750 4400 50  0001 L CNN
 F 3 "~" H 1700 4600 50  0001 C CNN
 F 4 "https://www.digikey.com/product-detail/en/advanced-photonix/NSL-5910/NSL-5910-ND/5436028" H 1700 4650 50  0001 C CNN "Part URL"
@@
 F 0 "R14" V 1400 5800 50  0000 C CNN
 F 1 "R_PHOTO" V 1491 5800 50  0000 C CNN
-F 2 "Connector_PinHeader_1.00mm:PinHeader_1x02_P1.00mm_Vertical" V 1775 5550 50  0001 L CNN
+F 2 "Custom:PinHeader_1x02_P1.00mm_Vertical" V 1775 5550 50  0001 L CNN
 F 3 "~" H 1725 5750 50  0001 C CNN
 F 4 "https://www.digikey.com/product-detail/en/advanced-photonix/NSL-5910/NSL-5910-ND/5436028" H 1725 5800 50  0001 C CNN "Part URL"
@@
 F 0 "R15" V 1425 6950 50  0000 C CNN
 F 1 "R_PHOTO" V 1516 6950 50  0000 C CNN
-F 2 "Connector_PinHeader_1.00mm:PinHeader_1x02_P1.00mm_Vertical" V 1800 6700 50  0001 L CNN
+F 2 "Custom:PinHeader_1x02_P1.00mm_Vertical" V 1800 6700 50  0001 L CNN
 F 3 "~" H 1750 6900 50  0001 C CNN
 F 4 "https://www.digikey.com/product-detail/en/advanced-photonix/NSL-5910/NSL-5910-ND/5436028" H 1750 6950 50  0001 C CNN "Part URL"
@@
 NoConn ~ 4775 4725
 NoConn ~ 4775 4825
-NoConn ~ 3200 5400
 Wire Wire Line
 	10625 4350 10850 4350
@@
 Text Label 10850 5450 0    50   ~ 0
 IN2
+Wire Wire Line
+	2725 3250 3150 3250
+Wire Wire Line
+	3650 3150 4050 3150
+Wire Wire Line
+	3650 3350 3850 3350
 $EndSCHEMATC
