File: Circuitry/Joe/Joe.kicad_pcb (KiCad board)
At the start: 2 copper layers, 51.1 x 107.3 mm, 32 parts, among them J1 Conn_02x03_Counter_Clockwise, J2 Conn_01x20, J3 USB_B_Micro, J4 Micro_SD_Card, U5 DS3231MZ, U6 M24C32-XDW5TP, U7 NSL BUS, U8 AP2127N-3.3, U9 ATmega32U4-MU

Commit message: planet on pcb!
Parts:
- added G***: LOGO, Custom:planet, F.Cu at (-12.2, -31.7)
Changed lines of the file:
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@@
-(kicad_pcb (version 20171130) (host pcbnew "(5.1.2)-2")
+(kicad_pcb (version 20171130) (host pcbnew 5.1.2-f72e74a~84~ubuntu18.04.1)
   (general
     (thickness 1.6)
@@
     (tracks 646)
     (zones 0)
-    (modules 32)
+    (modules 33)
     (nets 61)
   )
   (page A4)
   (layers
-    (0 F.Cu signal)
-    (31 B.Cu signal)
+    (0 F.Cu signal hide)
+    (31 B.Cu signal hide)
     (32 B.Adhes user)
     (33 F.Adhes user)
@@
     (add_net "Net-(U9-Pad16)")
   )
+  (module Custom:planet (layer F.Cu)
+    (at -12.2428 -31.6992 90)
+    (fp_text reference G*** (at 0 0 90) (layer F.SilkS) hide
+      (effects (font (size 1.524 1.524) (thickness 0.3)))
+    )
+    (fp_text value LOGO (at 0.75 0 90) (layer F.SilkS) hide
+      (effects (font (size 1.524 1.524) (thickness 0.3)))
+    )
+    (fp_poly (pts (xy 7.446063 -9.400031) (xy 7.984328 -9.266004) (xy 8.410346 -9.069448) (xy 8.777817 -8.781538)
+      (xy 8.964748 -8.58484) (xy 9.202293 -8.273722) (xy 9.371917 -7.941141) (xy 9.482981 -7.552285)
+      (xy 9.544847 -7.072337) (xy 9.566876 -6.466484) (xy 9.567333 -6.343902) (xy 9.543394 -5.66664)
+      (xy 9.465668 -5.021627) (xy 9.325294 -4.378594) (xy 9.113411 -3.707273) (xy 8.821156 -2.977396)
+      (xy 8.439669 -2.158693) (xy 8.205687 -1.692886) (xy 7.981756 -1.253245) (xy 7.823706 -0.928293)
+      (xy 7.72006 -0.682089) (xy 7.659341 -0.478693) (xy 7.63007 -0.282162) (xy 7.620772 -0.056555)
+      (xy 7.62 0.141166) (xy 7.537224 1.21288) (xy 7.294609 2.278877) (xy 6.900724 3.315761)
+      (xy 6.364136 4.300135) (xy 5.819926 5.056339) (xy 5.080162 5.835777) (xy 4.219029 6.502041)
+      (xy 3.246838 7.048426) (xy 2.173895 7.468224) (xy 2.057111 7.504295) (xy 1.690527 7.605739)
+      (xy 1.353287 7.674034) (xy 0.990854 7.716337) (xy 0.548691 7.739807) (xy 0.198528 7.748253)
+      (xy -0.915277 7.767705) (xy -1.934075 8.287119) (xy -2.421057 8.522163) (xy -2.962329 8.762235)
+      (xy -3.486931 8.976884) (xy -3.868269 9.117124) (xy -4.283589 9.252885) (xy -4.61746 9.344027)
+      (xy -4.929295 9.400704) (xy -5.278507 9.433067) (xy -5.724508 9.451269) (xy -5.842 9.454393)
+      (xy -6.452658 9.45762) (xy -6.906414 9.431979) (xy -7.213328 9.376855) (xy -7.239 9.368818)
+      (xy -7.945053 9.06648) (xy -8.510724 8.671085) (xy -8.940915 8.176557) (xy -9.240529 7.576824)
+      (xy -9.414467 6.865813) (xy -9.416675 6.847624) (xy 0.550334 6.847624) (xy 0.889 6.801528)
+      (xy 1.165383 6.75423) (xy 1.51115 6.682314) (xy 1.730769 6.630849) (xy 2.628314 6.324744)
+      (xy 3.486778 5.87029) (xy 4.283007 5.287724) (xy 4.993849 4.59728) (xy 5.596153 3.819193)
+      (xy 6.066766 2.973698) (xy 6.158249 2.761268) (xy 6.26114 2.483738) (xy 6.371056 2.148416)
+      (xy 6.477195 1.794074) (xy 6.568751 1.459486) (xy 6.634921 1.183426) (xy 6.664902 1.004665)
+      (xy 6.660312 0.959423) (xy 6.600165 1.010075) (xy 6.458697 1.169254) (xy 6.257881 1.411307)
+      (xy 6.049975 1.671919) (xy 5.451768 2.384258) (xy 4.73103 3.158466) (xy 3.911832 3.971664)
+      (xy 3.018244 4.800976) (xy 2.074337 5.623522) (xy 1.10418 6.416425) (xy 0.844061 6.619979)
+      (xy 0.550334 6.847624) (xy -9.416675 6.847624) (xy -9.441954 6.639457) (xy -9.448728 5.860446)
+      (xy -9.369747 5.276773) (xy -6.234421 5.276773) (xy -6.2235 5.500059) (xy -6.212072 5.563437)
+      (xy -6.060887 5.934911) (xy -5.816314 6.174744) (xy -5.467003 6.289673) (xy -5.001601 6.286438)
+      (xy -4.995333 6.285717) (xy -4.759455 6.253076) (xy -4.605731 6.22196) (xy -4.57937 6.211387)
+      (xy -4.620579 6.143387) (xy -4.759534 5.983744) (xy -4.972476 5.758758) (xy -5.153422 5.575891)
+      (xy -5.430025 5.291123) (xy -5.673444 5.022806) (xy -5.848935 4.810086) (xy -5.90514 4.728909)
+      (xy -6.017448 4.564177) (xy -6.098979 4.487959) (xy -6.103347 4.487334) (xy -6.151623 4.563166)
+      (xy -6.193129 4.755341) (xy -6.222513 5.010872) (xy -6.234421 5.276773) (xy -9.369747 5.276773)
+      (xy -9.332852 5.004118) (xy -9.103399 4.099562) (xy -8.769444 3.175865) (xy -8.340063 2.262115)
+      (xy -7.824331 1.387401) (xy -7.784769 1.327693) (xy -7.626739 1.083921) (xy -7.528508 0.893526)
+      (xy -7.475822 0.70227) (xy -7.454429 0.455915) (xy -7.450076 0.100221) (xy -7.450027 0.053852)
+      (xy -7.446279 0) (xy -6.473793 0) (xy -6.47267 0.522552) (xy -6.465637 0.914586)
+      (xy -6.447798 1.214917) (xy -6.414259 1.462357) (xy -6.360122 1.695721) (xy -6.280494 1.95382)
+      (xy -6.196136 2.201334) (xy -5.796056 3.160681) (xy -5.29588 4.001479) (xy -4.815667 4.60462)
+      (xy -4.498444 4.936769) (xy -4.172285 5.241601) (xy -3.866162 5.495407) (xy -3.609044 5.674476)
+      (xy -3.429901 5.755101) (xy -3.407189 5.757334) (xy -3.277871 5.718779) (xy -3.041194 5.615302)
+      (xy -2.737286 5.465179) (xy -2.559181 5.371062) (xy -1.075365 4.485276) (xy 0.320175 3.484036)
+      (xy 1.611072 2.381922) (xy 2.780958 1.193511) (xy 3.813464 -0.066615) (xy 4.265532 -0.70771)
+      (xy 4.504892 -1.08178) (xy 4.759601 -1.50702) (xy 5.014401 -1.954741) (xy 5.254036 -2.396256)
+      (xy 5.463248 -2.802875) (xy 5.62678 -3.145912) (xy 5.729376 -3.396678) (xy 5.757334 -3.512777)
+      (xy 5.699013 -3.695331) (xy 5.53763 -3.965573) (xy 5.293552 -4.295265) (xy 4.987144 -4.656168)
+      (xy 4.752086 -4.906525) (xy 4.260251 -5.34735) (xy 3.67231 -5.778063) (xy 3.057292 -6.151079)
+      (xy 2.69676 -6.329203) (xy 4.573849 -6.329203) (xy 5.150598 -5.795222) (xy 5.435464 -5.519549)
+      (xy 5.695042 -5.247415) (xy 5.88622 -5.024721) (xy 5.930098 -4.965344) (xy 6.065626 -4.791256)
+      (xy 6.165946 -4.704416) (xy 6.187006 -4.702917) (xy 6.227381 -4.79939) (xy 6.270257 -5.008291)
+      (xy 6.29074 -5.155006) (xy 6.297424 -5.652268) (xy 6.185671 -6.028565) (xy 5.955901 -6.283542)
+      (xy 5.608536 -6.416845) (xy 5.143995 -6.428118) (xy 4.837508 -6.381935) (xy 4.573849 -6.329203)
+      (xy 2.69676 -6.329203) (xy 2.667 -6.343906) (xy 1.799652 -6.640248) (xy 0.861562 -6.807853)
+      (xy -0.108012 -6.846721) (xy -1.06981 -6.756853) (xy -1.984571 -6.538248) (xy -2.497666 -6.343906)
+      (xy -3.386263 -5.861739) (xy -4.196541 -5.239426) (xy -4.913278 -4.493961) (xy -5.521252 -3.642335)
+      (xy -6.005239 -2.701544) (xy -6.189104 -2.223106) (xy -6.294581 -1.910323) (xy -6.370108 -1.655798)
+      (xy -6.420694 -1.420413) (xy -6.451349 -1.165049) (xy -6.467082 -0.850589) (xy -6.472903 -0.437914)
+      (xy -6.473793 0) (xy -7.446279 0) (xy -7.369861 -1.0979) (xy -7.136816 -2.205637)
+      (xy -6.759172 -3.255166) (xy -6.245209 -4.232289) (xy -5.603206 -5.122811) (xy -4.841445 -5.912536)
+      (xy -3.968205 -6.587269) (xy -3.367642 -6.945267) (xy -2.456787 -7.355571) (xy -1.510861 -7.625406)
+      (xy -0.499529 -7.761692) (xy 0.296334 -7.780844) (xy 0.727126 -7.775195) (xy 1.029327 -7.779792)
+      (xy 1.243652 -7.801802) (xy 1.410815 -7.848386) (xy 1.57153 -7.926711) (xy 1.75653 -8.03779)
+      (xy 2.424543 -8.39811) (xy 3.181097 -8.719119) (xy 3.991578 -8.992529) (xy 4.821369 -9.210053)
+      (xy 5.635857 -9.363403) (xy 6.400426 -9.444291) (xy 7.080461 -9.444429) (xy 7.446063 -9.400031)) (layer B.SilkS) (width 0.01))
+  )
   (module "" (layer F.Cu)

Commit message: Build zip for joe
Parts:
- R12: value P1 -> R_PHOTO; footprint Custom:PinHeader_1x02_P1.00mm_Vertical -> Connector_PinHeader_2.00mm:PinHeader_1x02_P2.00mm_Vertical
- R13: value P3 -> R_PHOTO; footprint Custom:PinHeader_1x02_P1.00mm_Vertical -> Connector_PinHeader_2.00mm:PinHeader_1x02_P2.00mm_Vertical; moved to F.Cu
- R14: value P3 -> R_PHOTO; footprint Custom:PinHeader_1x02_P1.00mm_Vertical -> Connector_PinHeader_2.00mm:PinHeader_1x02_P2.00mm_Vertical
- R15: value P4 -> R_PHOTO; footprint Custom:PinHeader_1x02_P1.00mm_Vertical -> Connector_PinHeader_2.00mm:PinHeader_1x02_P2.00mm_Vertical
- U7: value NSL BUS -> DF12-20DS
- moved R3 5.18 mm to (-43.0, 27.5), turned to 270 degrees
- moved R5 2.02 mm to (-42.9, 30.9)
- moved R12 1.81 mm to (-47.7, 33.9)
- moved R1 1.38 mm to (-42.9, 34.3)
- moved R15 0.87 mm to (-47.8, 30.4)
- turned R13 to 90 degrees
Routing:
- net GND: track 93.2 -> 90.3 mm, vias 24 -> 23
- net /PHO2: track 62.3 -> 60.2 mm
- net +3V3: track 108.2 -> 109.6 mm
- net /PHO4: track 55.3 -> 55.9 mm
- net /PHO1: track 61.9 -> 61.4 mm
