File: Circuitry/Bill/Bill.sch (KiCad schematic (older format))
At the start: 16 parts, among them U1 DS3231M

Commit message: sch review changes, eeprom, linear image sensor.
Parts:
- removed R? (x4): R_10K, footprints:R_0805_OEM, symbol RTC_Circuit-rescue:R_10K-formula
- added R? (x4): R, symbol Device:R
Connections:
- wire segments 51 -> 54
Changed lines of the file:
@@
-	1    0    0    -1
-$EndComp
-$Comp
-L RTC_Circuit-rescue:R_10K-formula R?
-U 1 1 5D03BEF7
-P 1150 1400
-F 0 "R?" H 1220 1446 50  0000 L CNN
-F 1 "R_10K" H 1220 1355 50  0000 L CNN
-F 2 "footprints:R_0805_OEM" H 1080 1400 50  0001 C CNN
-F 3 "http://www.bourns.com/data/global/pdfs/CRS.pdf" H 1230 1400 50  0001 C CNN
-F 4 "DK" H 1150 1400 60  0001 C CNN "MFN"
-F 5 "CRS0805-FX-1002ELFCT-ND" H 1150 1400 60  0001 C CNN "MPN"
-F 6 "https://www.digikey.com/products/en?keywords=CRS0805-FX-1002ELFCT-ND" H 1630 1800 60  0001 C CNN "PurchasingLink"
-	1    1150 1400
-	1    0    0    -1
-$EndComp
-$Comp
-L RTC_Circuit-rescue:R_10K-formula R?
-U 1 1 5D03BF79
-P 1000 1300
-F 0 "R?" H 800 1375 50  0000 L CNN
-F 1 "R_10K" H 675 1275 50  0000 L CNN
-F 2 "footprints:R_0805_OEM" H 930 1300 50  0001 C CNN
-F 3 "http://www.bourns.com/data/global/pdfs/CRS.pdf" H 1080 1300 50  0001 C CNN
-F 4 "DK" H 1000 1300 60  0001 C CNN "MFN"
-F 5 "CRS0805-FX-1002ELFCT-ND" H 1000 1300 60  0001 C CNN "MPN"
-F 6 "https://www.digikey.com/products/en?keywords=CRS0805-FX-1002ELFCT-ND" H 1480 1700 60  0001 C CNN "PurchasingLink"
-	1    1000 1300
 	1    0    0    -1
 $EndComp
@@
 Wire Wire Line
 	1450 1850 725  1850
-$Comp
-L RTC_Circuit-rescue:R_10K-formula R?
-U 1 1 5D11A655
-P 2750 1450
-F 0 "R?" H 2575 1525 50  0000 L CNN
-F 1 "R_10K" H 2450 1400 50  0000 L CNN
-F 2 "footprints:R_0805_OEM" H 2680 1450 50  0001 C CNN
-F 3 "http://www.bourns.com/data/global/pdfs/CRS.pdf" H 2830 1450 50  0001 C CNN
-F 4 "DK" H 2750 1450 60  0001 C CNN "MFN"
-F 5 "CRS0805-FX-1002ELFCT-ND" H 2750 1450 60  0001 C CNN "MPN"
-F 6 "https://www.digikey.com/products/en?keywords=CRS0805-FX-1002ELFCT-ND" H 3230 1850 60  0001 C CNN "PurchasingLink"
-	1    2750 1450
-	1    0    0    -1
-$EndComp
-$Comp
-L RTC_Circuit-rescue:R_10K-formula R?
-U 1 1 5D11A65E
-P 2975 1300
-F 0 "R?" H 3075 1375 50  0000 L CNN
-F 1 "R_10K" H 3075 1275 50  0000 L CNN
-F 2 "footprints:R_0805_OEM" H 2905 1300 50  0001 C CNN
-F 3 "http://www.bourns.com/data/global/pdfs/CRS.pdf" H 3055 1300 50  0001 C CNN
-F 4 "DK" H 2975 1300 60  0001 C CNN "MFN"
-F 5 "CRS0805-FX-1002ELFCT-ND" H 2975 1300 60  0001 C CNN "MPN"
-F 6 "https://www.digikey.com/products/en?keywords=CRS0805-FX-1002ELFCT-ND" H 3455 1700 60  0001 C CNN "PurchasingLink"
-	1    2975 1300
-	1    0    0    -1
-$EndComp
 Wire Wire Line
 	2450 1750 2750 1750
@@
 	8775 5525 11175 5525
 Wire Wire Line
-	725  1450 1450 1450
-Wire Wire Line
-	725  1550 1450 1550
-Wire Wire Line
-	2450 1450 3250 1450
+	725  1450 1000 1450
+Wire Wire Line
+	725  1550 1150 1550
+Wire Wire Line
+	2450 1450 2975 1450
+$Comp
+L Device:R R?
+U 1 1 5D1912DB
+P 1000 1300
+F 0 "R?" H 825 1375 50  0000 L CNN
+F 1 "R" H 825 1300 50  0000 L CNN
+F 2 "" V 930 1300 50  0001 C CNN
+F 3 "~" H 1000 1300 50  0001 C CNN
+	1    1000 1300
+	1    0    0    -1
+$EndComp
+Connection ~ 1000 1450
+Wire Wire Line
+	1000 1450 1450 1450
+$Comp
+L Device:R R?
+U 1 1 5D19223D
+P 1150 1400
+F 0 "R?" H 1220 1446 50  0000 L CNN
+F 1 "R" H 1220 1355 50  0000 L CNN
+F 2 "" V 1080 1400 50  0001 C CNN
+F 3 "~" H 1150 1400 50  0001 C CNN
+	1    1150 1400
+	1    0    0    -1
+$EndComp
+Connection ~ 1150 1550
+Wire Wire Line
+	1150 1550 1450 1550
+$Comp
+L Device:R R?
+U 1 1 5D194B82
+P 2750 1450
+F 0 "R?" H 2820 1496 50  0000 L CNN
+F 1 "R" H 2820 1405 50  0000 L CNN
+F 2 "" V 2680 1450 50  0001 C CNN
+F 3 "~" H 2750 1450 50  0001 C CNN
+	1    2750 1450
+	1    0    0    -1
+$EndComp
+$Comp
+L Device:R R?
+U 1 1 5D195CC5
+P 2975 1300
+F 0 "R?" H 3045 1346 50  0000 L CNN
+F 1 "R" H 3045 1255 50  0000 L CNN
+F 2 "" V 2905 1300 50  0001 C CNN
+F 3 "~" H 2975 1300 50  0001 C CNN
+	1    2975 1300
+	1    0    0    -1
+$EndComp
+Connection ~ 2975 1450
+Wire Wire Line
+	2975 1450 3250 1450
 $EndSCHEMATC

Commit message: bill schematic
Parts:
- removed U?: DF12-20DS, symbol Custom:DF12-20DS
- added C3, C4: 1uF, symbol Device:C_Small
- added U2: UFDFPN8-MC-Custom, symbol Custom:UFDFPN8-MC-Custom
- added U3: DF12-20DS-Custom, symbol Custom:DF12-20DS-Custom
- C1: renamed from C?; value CP_Small -> 0.1uF
- C2: renamed from C?; value C_Small -> 0.1uF
- R1, R2, R3, R4: renamed from R?; value R -> 10k
- gave numbers to parts that had none: 8
Connections:
- net 3.3V: now also U3.18 (3.3V)
- net 5V: now also U3.17 (5V)
- net BUSY: now also U3.13 (BUSY); no longer D1.2 (A)
- net GND: now also J1.6 (Pin_6), U4.5 (UGND), C3.1, C4.1, U2.1 (E0), U2.2 (E1), U2.3 (E2), U2.4 (Vss), U3.19 (GND), U3.20 (GND); no longer J1.4 (Pin_4)
- net MOSI: now also J1.4 (Pin_4); no longer J1.5 (Pin_5)
- net RST: now also J1.5 (Pin_5); no longer J1.3 (Pin_3)
- net RX: now also U4.21 (PD3), U3.11 (RX)
- net SCK: now also J1.3 (Pin_3); no longer J1.2 (Pin_2)
- net SDA: now also U2.5 (SDA)
- net SQW: no longer D2.2 (A)
- net TX: now also U4.20 (PD2), U3.12 (TX)
- net SCL: now reaches U4.18 (PD0)
- net SCL: now also U2.6 (SCL)
- net VBUS: now reaches U4.2 (UVCC)
- net VBUS: now also U4.7 (VBUS)
- net PLED2: now reaches U4.29 (PB5)
- net PLED2: now also D2.2 (A)
- net PLED3: now reaches U4.30 (PB6)
- net PLED3: now also D3.2 (A)
- net WC: now reaches U4.41 (PF0)
- net WC: now also U2.7 (WC)
- net at U4.42 (AREF): now also C3.2
- net at U4.6 (UCAP): now also C4.2
- net +5V renamed +3V3
- net +3V3: now also J1.2 (Pin_2), U2.8 (Vcc); no longer J1.6 (Pin_6)
- net PHOV renamed PLED1
- net PLED1: now also D1.2 (A)
- net TEMPV: no longer names the net of U4.27 (PD7)
- no-connect marks 1 -> 30
Other:
- note added: "EEPROM"
- moved on the sheet: D1, D2, D3, R5, R6, R7
